Commit message: xacro basarili calisti

File: arm3dof/models/arm3dof/model.urdf.xacro (robot description, xacro)
@@ -1,7 +1,4 @@
 <?xml version="1.0" ?>
 <robot xmlns:xacro="http://www.ros.org/wiki/xacro"
-    xmlns:sensor="http://playerstage.sourceforge.net/gazebo/xmlschema/#sensor"
-    xmlns:controller="http://playerstage.sourceforge.net/gazebo/xmlschema/#controller"
-    xmlns:interface="http://playerstage.sourceforge.net/gazebo/xmlschema/#interface"
     name="arm3dof">
   <xacro:property name="base_width" value="0.9" />
@@ -13,8 +10,10 @@
   <xacro:macro name="box_inertia" params="m w h d">
     <inertial>
+      <origin xyz="0 0 ${h / 2}" rpy="0 0 0" />
       <mass value="${m}" />
-      <inertia ixx="${(m/12) * (h*h + d*d)}" ixy="0.0" ixz="0.0"
-      iyy="${(m/12) * (w*w + d*d)}" iyz="0.0"
-      izz="${(m/12) * (w*w + h*h)}" />
+      <inertia
+      ixx="${(m/12) * (h*h + d*d)}" ixy="0.0" ixz="0.0"
+      iyy="${(m/12) * (w*w + h*h)}" iyz="0.0"
+      izz="${(m/12) * (w*w + d*d)}" />
     </inertial>
   </xacro:macro>
@@ -33,5 +32,5 @@
         <origin xyz="0 0 ${link_length / 2}" rpy="0 0 0" />
         <geometry>
-          <box size="${link_width} ${link_width} ${link_length}" />
+          <box size="${link_width} ${link_width} ${link_length - 0.05}" />
         </geometry>
       </collision>
@@ -80,8 +79,8 @@
     <parent link="base_link" />
     <child link="link_1" />
-    <origin xyz="0 0 ${base_height / 2}" rpy="0 0 0" />
+    <origin xyz="0 0 ${base_height}" rpy="0 0 0" />
     <axis xyz="0 0 1" />
     <limit lower="-3.14" upper="3.14" effort="100" velocity="10" />
-    <dynamics damping="0.5"/>
+    <dynamics damping="3.0" friction="1.0"/>
   </joint>
   <xacro:arm_link link_name="link_1" color_name="blue" color_rgb="0 0 0.8 1" />
@@ -92,5 +91,5 @@
     <axis xyz="0 1 0" />
     <limit lower="-1.57" upper="1.57" effort="100" velocity="10" />
-    <dynamics damping="0.5"/>
+    <dynamics damping="3.0" friction="1.0"/>
   </joint>
   <xacro:arm_link link_name="link_2" color_name="red" color_rgb="0.5 0 0 1" />
@@ -101,5 +100,5 @@
     <axis xyz="0 1 0" />
     <limit lower="-1.57" upper="1.57" effort="100" velocity="10" />
-    <dynamics damping="0.5"/>
+    <dynamics damping="3.0" friction="1.0"/>
   </joint>
   <xacro:arm_link link_name="link_3" color_name="blue" color_rgb="0 0 0.8 1" />
@@ -109,5 +108,5 @@
       <topic>cmd_pos_j1</topic>
       <p_gain>200</p_gain>
-      <i_gain>10</i_gain>
+      <i_gain>1</i_gain>
       <d_gain>10</d_gain>
     </plugin>
@@ -115,6 +114,6 @@
       <joint_name>j2_base_shoulder</joint_name>
       <topic>cmd_pos_j2</topic>
-      <p_gain>5000</p_gain>
-      <i_gain>200</i_gain>
+      <p_gain>1000</p_gain>
+      <i_gain>1</i_gain>
       <d_gain>50</d_gain>
     </plugin>
@@ -122,6 +121,6 @@
       <joint_name>j3_base_elbow</joint_name>
       <topic>cmd_pos_j3</topic>
-      <p_gain>1000</p_gain>
-      <i_gain>50</i_gain>
+      <p_gain>500</p_gain>
+      <i_gain>1</i_gain>
       <d_gain>20</d_gain>
     </plugin>
